Commit message: Add Kinect sensor to Robocup version of REEM.
- Patch provided by Jose Capriles.

File: reem_robocup_description/robots/reem_robocup.urdf.xacro (robot description, xacro)
@@ -25,4 +25,6 @@
   <!-- Camera sensors -->
   <include filename="$(find reem_description)/urdf/sensors/stereo_camera.urdf.xacro" />
+  <!-- Kinect -->
+  <include filename="$(find reem_description)/urdf/sensors/kinect.urdf.xacro" />
   <!-- Generic simulator_gazebo plugins -->
   <include filename="$(find reem_description)/gazebo/gazebo.urdf.xacro" />
@@ -45,3 +47,7 @@
     <origin xyz="0.08203  -0.09558  0.04132" rpy="1.56293 -0.00855922 -0.0201307" />
   </xacro:stereo_camera_v0>
+  <!-- kinect camera -->
+  <xacro:kinect_v0 parent="head_2_link" name="kinect">
+     <origin xyz="0.0 0.0 0.45" rpy="0.0 0.0 0.0" />
+  </xacro:kinect_v0>
 </robot>
